File: CannedPIHat.kicad_sch (KiCad schematic)
At the start: 103 parts, among them IC1 TPS56428DDA, IC2 LM1117MPX-3.3, IC3 STM32G474RET6, IC4 TJA1021TK_20_C,118, IC6 SN74LVC1G66QDCKRQ1, IC7 SN74LVC1G66QDCKRQ1, IC8 SN74LVC1G66QDCKRQ1, J1 Barrel_Jack_Switch, J2 09562627813, J5 20021511-00014T4LF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

Commit message: Update to Rev C.
Parts:
- removed IC2: LM1117MPX-3.3, Package_TO_SOT_SMD:SOT-223, symbol SamacSys_Parts:LM1117MPX-3.3
- removed R9: 0R, Resistor_SMD:R_0402_1005Metric, symbol Device:R_US
- added C18, C22: DNP, Capacitor_SMD:C_0402_1005Metric, symbol Device:C
- added C35: 0.1uF, Capacitor_SMD:C_0603_1608Metric, symbol Device:C
- added U6: AP2112K-3.3, Package_TO_SOT_SMD:SOT-23-5, symbol Regulator_Linear:AP2112K-3.3
- added Y2: 8Mhz, Crystal:Crystal_SMD_3225-4Pin_3.2x2.5mm, symbol Device:Crystal_GND24
- BT1: Digi-Key_PN (none) -> 952-1745-1-ND; Manufacturer_Part_Number (none) -> S8411-45R
- C1: Digi-Key_PN (none) -> 565-2549-1-ND; Manufacturer_Part_Number (none) -> EMZA250ADA101MF80G
- C10, C11, C13, C15, C16, C19, C2, C20, C21, C26, C27, C29, C30, C32, C33, C34, C7, C9: Digi-Key_PN (none) -> 311-1341-1-ND; Manufacturer_Part_Number (none) -> CC0603KRX7R8BB104
- C12, C14: Digi-Key_PN (none) -> 490-5949-1-ND; Manufacturer_Part_Number (none) -> GRM1555C1H6R8CA01D
- C17, C8: Digi-Key_PN (none) -> 587-3328-1-ND; Manufacturer_Part_Number (none) -> EMK316ABJ226ML-T
- C23, C28, C31: Digi-Key_PN (none) -> 587-4280-1-ND; Manufacturer_Part_Number (none) -> JMK212BBJ476MG-T
- C24: Digi-Key_PN (none) -> 311-1073-1-ND; Manufacturer_Part_Number (none) -> CC0603JRNPO9BN221
- C3: Digi-Key_PN (none) -> 1276-3107-1-ND; Manufacturer_Part_Number (none) -> CL31B106KQHNFNE
- C4: value 0.1uF -> 1uF; Digi-Key_PN (none) -> 311-1341-1-ND; Manufacturer_Part_Number (none) -> CC0603KRX7R8BB104
- C5: value 0.1uF -> 2uF; Digi-Key_PN (none) -> 311-1341-1-ND; Manufacturer_Part_Number (none) -> CC0603KRX7R8BB104
- C6: Digi-Key_PN (none) -> 445-5810-1-ND; Manufacturer_Part_Number (none) -> CGA3E2X7R2A472K080AA
- CR1: Digi-Key_PN (none) -> 1727-1225-1-ND; Manufacturer_Part_Number (none) -> PESD1LIN,135
- D1: Digi-Key_PN (none) -> S1GFSCT-ND; Manufacturer_Part_Number (none) -> S1G
- D10: Digi-Key_PN (none) -> 475-2815-1-ND; Manufacturer_Part_Number (none) -> LB Q39E-N1OO-35-1
- D11: Digi-Key_PN (none) -> 475-3754-1-ND; Manufacturer_Part_Number (none) -> LG Q396-PS-35
- D12, D13, D3, D4: Digi-Key_PN (none) -> 475-2512-1-ND; Manufacturer_Part_Number (none) -> LS Q976-NR-1
- D2: Digi-Key_PN (none) -> SMBJ36CA-FDICT-ND; Manufacturer_Part_Number (none) -> SMBJ36CA-13-F
- D5, D8, D9: Manufacturer_Part_Number (none) -> PESD2CAN,215
- D6: Digi-Key_PN (none) -> 1N4448WXTPMSCT-ND; Manufacturer_Part_Number (none) -> ‎1N4448WX-TP‎
- F1: Digi-Key_PN (none) -> 507-1812-1-ND; Manufacturer_Part_Number (none) -> 0ZCK0035FF2G
- IC1: Digi-Key_PN (none) -> 296-35856-1-ND
- IC3: Digi-Key_PN (none) -> 497-STM32G474RET6-ND
- J2: Digi-Key_PN (none) -> L717HDA26PD1CH4F-ND
- J5: Digi-Key_PN (none) -> 612-FTSH-107-01-L-D-K-ND
- J6: Digi-Key_PN (none) -> 2073-USB4085-GF-ACT-ND; Manufacturer_Part_Number (none) -> USB4085-GF-A
- P1: Digi-Key_PN (none) -> 952-3230-2-ND; Manufacturer_Part_Number (none) -> M20-7812045R
- R1, R16, R26, R31: Digi-Key_PN (none) -> 311-10.0KHRCT-ND; Manufacturer_Part_Number (none) -> RC0603FR-0710KL
- R12: Digi-Key_PN (none) -> 311-4.7KGRCT-ND; Manufacturer_Part_Number (none) -> RC0603JR-074K7L
- R17: Digi-Key_PN (none) -> 311-33.2KHRCT-ND; Manufacturer_Part_Number (none) -> RC0603FR-0733K2L
- R19, R21, R22, R23, R25, R30, R35, R36, R5, R7: Digi-Key_PN (none) -> 311-1.00KHRCT-ND; Manufacturer_Part_Number (none) -> RC0603FR-071KL
- R2: Digi-Key_PN (none) -> 311-100KHRCT-ND; Manufacturer_Part_Number (none) -> RC0603FR-07100KL
- R20, R28, R34: Digi-Key_PN (none) -> 311-120HRCT-ND; Manufacturer_Part_Number (none) -> RC0603FR-07120RL
- R27, R29, R8: Digi-Key_PN (none) -> 311-0.0GRCT-ND; Manufacturer_Part_Number (none) -> RC0603JR-070RL
- R3: Digi-Key_PN (none) -> 13-AF0603FR-0749K9LCT-ND; Manufacturer_Part_Number (none) -> AF0603FR-0749K9L
- R32, R33: Digi-Key_PN (none) -> 311-5.1KGRCT-ND; Manufacturer_Part_Number (none) -> RC0603JR-075K1L
- R4: Digi-Key_PN (none) -> 13-AC0603FR-07365KLCT-ND; Manufacturer_Part_Number (none) -> 13-AC0603FR-07365KLCT-ND
- R6: value 0R -> 1k; footprint Resistor_SMD:R_0402_1005Metric -> Resistor_SMD:R_0603_1608Metric; Digi-Key_PN (none) -> 311-1.00KHRCT-ND; LCSC Part # C25741 -> C21190; Manufacturer_Part_Number (none) -> RC0603FR-071KL
- U4: Digi-Key_PN (none) -> 497-5235-1-ND; Manufacturer_Part_Number (none) -> USBLC6-2SC6
- Y1: value ECS-.327-6-12-C-TR -> 32.768Khz; footprint Crystal:Crystal_SMD_TXC_9HT11-2Pin_2.0x1.2mm -> Crystal:Crystal_SMD_2012-2Pin_2.0x1.2mm; Digi-Key_PN (none) -> XC2291CT-ND; Manufacturer_Part_Number (none) -> ECS-.327-6-12-C-TR
Connections:
- net +3V3: now also U6.5 (VOUT)
- net +5V: now also U6.1 (VIN), U6.3 (EN)
- net GND: now also J5.10 (Pin_10), C18.2, C22.2, C35.2, U6.2 (GND)
- net OSC32_IN: now also C12.1, Y1.1; no longer R6.1
- net OSC32_OUT: now also C14.1, Y1.2
- net RPI_3.3V: now reaches P1.1 (Pin_1)
- net RPI_3.3V: now also R6.1
- net RPI_SENSE: now reaches IC3.43 (PA9)
- net RPI_SENSE: now also R6.2, C35.1
- net OSC_IN: now reaches IC3.5 (PF0-OSC_IN)
- net OSC_IN: now also C18.1, Y2.1
- net OSC_OUT: now reaches IC3.6 (PF1-OSC_OUT)
- net OSC_OUT: now also C22.1, Y2.3
- no-connect marks 36 -> 33
Other:
- moved on the sheet: C12, C14, C4, C5
